Commit message: modify body collision

File: assets/urdf/a1/urdf/a1_old.urdf (robot description, URDF)
Before this commit: robot a1, 17 links, 16 joints
Links:
- link trunk: geometry collision box size=0.51 0.194 0.114; visual mesh filename=../meshes_old/trunk.dae scale=1 1 1

Commit message: debug

File: assets/urdf/a1/urdf/a1_old.urdf (robot description, URDF)
Before this commit: robot a1, 17 links, 16 joints
Links:
- link FL_hip: geometry collision cylinder length=0.04 radius=0.046; visual mesh filename=../meshes_old/hip.dae scale=1 1 1
- link FR_hip: geometry collision cylinder length=0.04 radius=0.046; visual mesh filename=../meshes_old/hip.dae scale=1 1 1
- link RL_hip: geometry collision cylinder length=0.04 radius=0.046; visual mesh filename=../meshes_old/hip.dae scale=1 1 1
- link RR_hip: geometry collision cylinder length=0.04 radius=0.046; visual mesh filename=../meshes_old/hip.dae scale=1 1 1
- link trunk: geometry collision box size=0.267 0.194 0.114; visual mesh filename=../meshes_old/trunk.dae scale=1 1 1
